File: PricklyPear/PricklyPear.sch (KiCad schematic (older format))
At the start: 4 parts, among them SW1 SW_SPDT

Commit message: Switch switch, add outline svg
Parts:
- SW1: footprint 1825232-1:1825232-1 -> Button_Switch_THT:SW_Slide_1P2T_CK_OS102011MS2Q
Changed lines of the file:
@@
 F 0 "SW1" H 7700 6535 50  0000 C CNN
 F 1 "SW_SPDT" H 7700 6444 50  0000 C CNN
-F 2 "1825232-1:1825232-1" H 7700 6250 50  0001 C CNN
+F 2 "Button_Switch_THT:SW_Slide_1P2T_CK_OS102011MS2Q" H 7700 6250 50  0001 C CNN
 F 3 "" H 7700 6250 50  0001 C CNN
 	1    7700 6250
